File: src/xchain.kicad_pcb (KiCad board)
At the start: 2 copper layers, 43.7 x 29.2 mm, 12 parts, among them Q1 PNP, Q2 PNP, SW1 SW_Push, SW2 SW_Push

Commit message: Revision
Routing:
- net Net-(D1-A): track 13.7 -> 55.6 mm, vias 0 -> 1
- net +3.3V: track 30.5 -> 64.0 mm
- net A: track 51.0 -> 52.1 mm
Changed lines of the file:
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@@
 			(psa4output no)
 			(plot_black_and_white yes)
-			(plotinvisibletext no)
 			(sketchpadsonfab no)
 			(plotpadnumbers no)
@@
 		(tags "Keystone type 3034 coin cell retainer")
 		(property "Reference" "BT1"
-			(at -8.525 7.2 315)
+			(at -10.4 7.3 315)
 			(layer "B.SilkS")
 			(effects
@@
 	)
 	(segment
+		(start 129.3 132.175)
+		(end 129.75 132.625)
+		(width 0.2)
+		(layer "F.Cu")
+		(net 1)
+	)
+	(segment
+		(start 155.325 132.9)
+		(end 152.975 135.25)
+		(width 0.2)
+		(layer "F.Cu")
+		(net 1)
+	)
+	(segment
+		(start 155.325 128.765)
+		(end 155.325 132.9)
+		(width 0.2)
+		(layer "F.Cu")
+		(net 1)
+	)
+	(segment
 		(start 141.55 139.05)
 		(end 140.075 140.525)
@@
 	)
 	(segment
+		(start 129.3 117.45)
+		(end 129.3 132.175)
+		(width 0.2)
+		(layer "F.Cu")
+		(net 1)
+	)
+	(segment
 		(start 131.275 140.525)
 		(end 129.3 138.55)
@@
 	)
 	(segment
+		(start 152.975 135.25)
+		(end 145.35 135.25)
+		(width 0.2)
+		(layer "F.Cu")
+		(net 1)
+	)
+	(segment
+		(start 145.35 135.25)
+		(end 141.55 139.05)
+		(width 0.2)
+		(layer "F.Cu")
+		(net 1)
+	)
+	(segment
 		(start 140.075 140.525)
 		(end 131.275 140.525)
@@
 		(net 1)
 	)
+	(via
+		(at 129.75 132.625)
+		(size 0.6)
+		(drill 0.3)
+		(layers "F.Cu" "B.Cu")
+		(net 1)
+	)
+	(segment
+		(start 129.75 132.625)
+		(end 129.75 138.1)
+		(width 0.2)
+		(layer "B.Cu")
+		(net 1)
+	)
+	(segment
+		(start 129.75 138.1)
+		(end 129.3 138.55)
+		(width 0.2)
+		(layer "B.Cu")
+		(net 1)
+	)
 	(segment
 		(start 149.62 139.5)
@@
 	)
 	(segment
-		(start 128.525 123.65)
-		(end 125.85 120.975)
+		(start 151.725 131.88)
+		(end 146.615 131.88)
 		(width 0.2)
 		(layer "F.Cu")
@@
 	)
 	(segment
-		(start 151.725 131.88)
-		(end 146.615 131.88)
+		(start 146.615 131.88)
+		(end 139.445 139.05)
 		(width 0.2)
 		(layer "F.Cu")
@@
 	)
 	(segment
-		(start 139.445 139.05)
-		(end 136.625 139.05)
+		(start 125.85 118.36)
+		(end 125.85 120.975)
 		(width 0.2)
 		(layer "F.Cu")
@@
 	)
 	(segment
-		(start 146.615 131.88)
-		(end 139.445 139.05)
+		(start 128.525 123.65)
+		(end 125.85 120.975)
 		(width 0.2)
 		(layer "F.Cu")
@@
 	)
 	(segment
-		(start 125.85 118.36)
-		(end 125.85 120.975)
+		(start 128.525 132.825)
+		(end 128.525 123.65)
 		(width 0.2)
 		(layer "F.Cu")
@@
 	)
 	(segment
-		(start 128.525 130.95)
-		(end 128.525 123.65)
+		(start 134.75 139.05)
+		(end 128.525 132.825)
 		(width 0.2)
 		(layer "F.Cu")
@@
 	)
 	(segment
-		(start 136.625 139.05)
-		(end 128.525 130.95)
+		(start 139.445 139.05)
+		(end 134.75 139.05)
 		(width 0.2)
 		(layer "F.Cu")
@@
 	(segment
 		(start 129.24 127.475)
+		(end 129.24 130.715)
+		(width 0.2)
+		(layer "B.Cu")
+		(net 7)
+	)
+	(segment
+		(start 129.24 127.475)
 		(end 127.85 127.475)
 		(width 0.2)
@@
 	)
 	(segment
+		(start 129.24 130.715)
+		(end 135.725 137.2)
+		(width 0.2)
+		(layer "B.Cu")
+		(net 7)
+	)
+	(segment
 		(start 127.855 127.475)
 		(end 125.855 129.475)
@@
 	)
 	(segment
+		(start 144.225 137.2)
+		(end 151.21 130.215)
+		(width 0.2)
+		(layer "B.Cu")
+		(net 7)
+	)
+	(segment
 		(start 127.85 127.475)
 		(end 125.85 125.475)
 		(width 0.2)
 		(layer "B.Cu")
+		(net 7)
+	)
+	(segment
+		(start 151.21 130.215)
+		(end 151.21 127.475)
+		(width 0.2)
+		(layer "B.Cu")
+		(net 7)
+	)
+	(segment
+		(start 135.725 137.2)
+		(end 144.225 137.2)
+		(width 0.2)
+		(layer "B.Cu")
